Commit message: finished assign5

File: ball.urdf (robot description, URDF)
Before this commit: robot robot, 1 links, 0 joints
Links:
- link Ball: geometry collision box size=1 1 1; visual box size=1 1 1

File: body.urdf (robot description, URDF)
Before this commit: robot robot, 3 links, 2 joints
Links:
- added link BackFlap, mass 1; collision box size=0.1 2 0.25; visual box size=0.1 2 0.25
- added link BackLeg1, mass 1; collision box size=1 0.7 1; visual box size=1 0.7 1
- link BackLeg: geometry collision box size=1 0.7 1; visual box size=1 0.7 1
Joints:
- added joint Torso_BackFlap: type revolute, parent Torso, child BackFlap, origin xyz=0.5 0 1.5 rpy=0 0 0, axis 0 1 0, limit lower=-3.14159 upper=3.14159 effort=0.0 velocity=0.0
- added joint Torso_BackLeg1: type revolute, parent Torso, child BackLeg1, origin xyz=0.5 0 1 rpy=0 0 0, axis 0 1 0, limit lower=-3.14159 upper=3.14159 effort=0.0 velocity=0.0
