Commit message: fixed names and added a sensor

File: body.urdf (robot description, URDF)
Before this commit: robot robot, 3 links, 2 joints
Links:
- removed link Link0
- removed link Link1
- removed link Link2
- added link BackLeg, mass 1; collision box size=1 1 1; visual box size=1 1 1
- added link FrontLeg, mass 1; collision box size=1 1 1; visual box size=1 1 1
- added link Torso, mass 1; collision box size=1 1 1; visual box size=1 1 1
Joints:
- removed joint Link0_Link1
- removed joint Link0_Link2
- added joint Torso_BackLeg: type revolute, parent Torso, child BackLeg, origin xyz=1 0 1 rpy=0 0 0, axis 0 1 0, limit lower=-3.14159 upper=3.14159 effort=0.0 velocity=0.0
- added joint Torso_FrontLeg: type revolute, parent Torso, child FrontLeg, origin xyz=2 0 1 rpy=0 0 0, axis 0 1 0, limit lower=-3.14159 upper=3.14159 effort=0.0 velocity=0.0

Commit message: progress in quad

File: body.urdf (robot description, URDF)
Before this commit: robot robot, 3 links, 2 joints
Links:
- link BackLeg: geometry collision box size=0.2 1 0.2; visual box size=0.2 1 0.2
- link FrontLeg: geometry collision box size=0.2 1 0.2; visual box size=0.2 1 0.2
Joints:
- joint Torso_BackLeg: axis 0 1 0 -> 1 0 0; origin xyz=1 0 1 rpy=0 0 0 -> xyz=0 -0.5 1 rpy=0 0 0
- joint Torso_FrontLeg: axis 0 1 0 -> 1 0 0; origin xyz=2 0 1 rpy=0 0 0 -> xyz=0 0.5 1 rpy=0 0 0

Commit message: done with quad

File: body.urdf (robot description, URDF)
Before this commit: robot robot, 3 links, 2 joints
Links:
- added link LeftLeg, mass 1; collision box size=1 0.2 0.2; visual box size=1 0.2 0.2
- added link LowerBackLeg, mass 1; collision box size=0.2 0.2 1; visual box size=0.2 0.2 1
- added link LowerFrontLeg, mass 1; collision box size=0.2 0.2 1; visual box size=0.2 0.2 1
- added link LowerLeftLeg, mass 1; collision box size=0.2 0.2 1; visual box size=0.2 0.2 1
- added link LowerRightLeg, mass 1; collision box size=0.2 0.2 1; visual box size=0.2 0.2 1
- added link RightLeg, mass 1; collision box size=1 0.2 0.2; visual box size=1 0.2 0.2
Joints:
- added joint BackLeg_LowerBackLeg: type revolute, parent BackLeg, child LowerBackLeg, origin xyz=0 -1 0 rpy=0 0 0, axis 1 0 0, limit lower=-3.14159 upper=3.14159 effort=0.0 velocity=0.0
- added joint FrontLeg_LowerFrontLeg: type revolute, parent FrontLeg, child LowerFrontLeg, origin xyz=0 1 0 rpy=0 0 0, axis 1 0 0, limit lower=-3.14159 upper=3.14159 effort=0.0 velocity=0.0
- added joint LeftLeg_LowerLeftLeg: type revolute, parent LeftLeg, child LowerLeftLeg, origin xyz=1 0 0 rpy=0 0 0, axis 0 1 0, limit lower=-3.14159 upper=3.14159 effort=0.0 velocity=0.0
- added joint Right_LowerRightLeg: type revolute, parent RightLeg, child LowerRightLeg, origin xyz=-1 0 0 rpy=0 0 0, axis 0 1 0, limit lower=-3.14159 upper=3.14159 effort=0.0 velocity=0.0
- added joint Torso_LeftLeg: type revolute, parent Torso, child LeftLeg, origin xyz=0.5 0 1 rpy=0 0 0, axis 0 1 0, limit lower=-3.14159 upper=3.14159 effort=0.0 velocity=0.0
- added joint Torso_RightLeg: type revolute, parent Torso, child RightLeg, origin xyz=-0.5 0 1 rpy=0 0 0, axis 0 1 0, limit lower=-3.14159 upper=3.14159 effort=0.0 velocity=0.0

Commit message: progress on assign 5

File: body.urdf (robot description, URDF)
Before this commit: robot robot, 9 links, 8 joints
Links:
- removed link LeftLeg
- removed link LowerBackLeg
- removed link LowerFrontLeg
- removed link LowerLeftLeg
- removed link LowerRightLeg
- removed link RightLeg
- link BackLeg: geometry collision box size=1 1 1; visual box size=1 1 1
- link FrontLeg: geometry collision box size=1 1 1; visual box size=1 1 1
- link Torso: geometry collision box size=2 2 0.5; visual box size=2 2 0.5
Joints:
- removed joint BackLeg_LowerBackLeg
- removed joint FrontLeg_LowerFrontLeg
- removed joint LeftLeg_LowerLeftLeg
- removed joint Right_LowerRightLeg
- removed joint Torso_LeftLeg
- removed joint Torso_RightLeg
- joint Torso_BackLeg: axis 1 0 0 -> 0 1 0; origin xyz=0 -0.5 1 rpy=0 0 0 -> xyz=0.5 0 1 rpy=0 0 0
- joint Torso_FrontLeg: axis 1 0 0 -> 0 1 0; origin xyz=0 0.5 1 rpy=0 0 0 -> xyz=2.5 0 1 rpy=0 0 0

Commit message: assign6 finished

File: body.urdf (robot description, URDF)
Before this commit: robot robot, 5 links, 4 joints
Links:
- removed link BackFlap
- removed link BackLeg
- removed link BackLeg1
- removed link FrontLeg
- removed link Torso
- added link Limb0, mass 1; collision box size=2.1 2.6 1.5; visual box size=2.1 2.6 1.5
- added link Limb1, mass 1; collision box size=1.7 2.4 2.0; visual box size=1.7 2.4 2.0
- added link Limb2, mass 1; collision box size=2.3 2.5 1.8; visual box size=2.3 2.5 1.8
- added link Limb3, mass 1; collision box size=1.8 2.6 2.3; visual box size=1.8 2.6 2.3
- added link Limb4, mass 1; collision box size=2.8 2.7 1.7; visual box size=2.8 2.7 1.7
- added link Limb5, mass 1; collision box size=2.9 2.4 2.1; visual box size=2.9 2.4 2.1
- added link Limb6, mass 1; collision box size=2.0 2.1 2.0; visual box size=2.0 2.1 2.0
- added link Limb7, mass 1; collision box size=2.0 2.8 2.0; visual box size=2.0 2.8 2.0
Joints:
- removed joint Torso_BackFlap
- removed joint Torso_BackLeg
- removed joint Torso_BackLeg1
- removed joint Torso_FrontLeg
- added joint Limb0_Limb1: type revolute, parent Limb0, child Limb1, origin xyz=0 0.375 0 rpy=0 0 0, axis 1 0 0, limit lower=-3.14159 upper=3.14159 effort=0.0 velocity=0.0
- added joint Limb1_Limb2: type revolute, parent Limb1, child Limb2, origin xyz=0 2.4 0 rpy=0 0 0, axis 1 0 0, limit lower=-3.14159 upper=3.14159 effort=0.0 velocity=0.0
- added joint Limb2_Limb3: type revolute, parent Limb2, child Limb3, origin xyz=0 2.5 0 rpy=0 0 0, axis 1 0 0, limit lower=-3.14159 upper=3.14159 effort=0.0 velocity=0.0
- added joint Limb3_Limb4: type revolute, parent Limb3, child Limb4, origin xyz=0 2.6 0 rpy=0 0 0, axis 1 0 0, limit lower=-3.14159 upper=3.14159 effort=0.0 velocity=0.0
- added joint Limb4_Limb5: type revolute, parent Limb4, child Limb5, origin xyz=0 2.7 0 rpy=0 0 0, axis 1 0 0, limit lower=-3.14159 upper=3.14159 effort=0.0 velocity=0.0
- added joint Limb5_Limb6: type revolute, parent Limb5, child Limb6, origin xyz=0 2.4 0 rpy=0 0 0, axis 1 0 0, limit lower=-3.14159 upper=3.14159 effort=0.0 velocity=0.0
- added joint Limb6_Limb7: type revolute, parent Limb6, child Limb7, origin xyz=0 2.1 0 rpy=0 0 0, axis 1 0 0, limit lower=-3.14159 upper=3.14159 effort=0.0 velocity=0.0

Commit message: assign6 finishedd

File: body.urdf (robot description, URDF)
Before this commit: robot robot, 8 links, 7 joints
Links:
- added link Limb10, mass 1; collision box size=2.0 2.6 2.9; visual box size=2.0 2.6 2.9
- added link Limb11, mass 1; collision box size=1.9 2.2 1.7; visual box size=1.9 2.2 1.7
- added link Limb12, mass 1; collision box size=1.9 1.5 1.7; visual box size=1.9 1.5 1.7
- added link Limb8, mass 1; collision box size=1.9 1.8 2.8; visual box size=1.9 1.8 2.8
- added link Limb9, mass 1; collision box size=2.9 1.6 2.8; visual box size=2.9 1.6 2.8
- link Limb0: geometry collision box size=2.1 1.8 1.8; visual box size=2.1 1.8 1.8
- link Limb1: geometry collision box size=2.5 2.6 2.0; visual box size=2.5 2.6 2.0
- link Limb2: geometry collision box size=2.0 1.9 1.7; visual box size=2.0 1.9 1.7
- link Limb3: geometry collision box size=2.7 2.0 1.7; visual box size=2.7 2.0 1.7
- link Limb4: geometry collision box size=1.5 2.9 2.6; visual box size=1.5 2.9 2.6
- link Limb5: geometry collision box size=2.5 1.5 2.0; visual box size=2.5 1.5 2.0
- link Limb6: geometry collision box size=2.2 2.8 2.7; visual box size=2.2 2.8 2.7
- link Limb7: geometry collision box size=2.5 2.4 2.5; visual box size=2.5 2.4 2.5
Joints:
- added joint Limb10_Limb11: type revolute, parent Limb10, child Limb11, origin xyz=0 2.6 0 rpy=0 0 0, axis 1 0 0, limit lower=-3.14159 upper=3.14159 effort=0.0 velocity=0.0
- added joint Limb11_Limb12: type revolute, parent Limb11, child Limb12, origin xyz=0 2.2 0 rpy=0 0 0, axis 1 0 0, limit lower=-3.14159 upper=3.14159 effort=0.0 velocity=0.0
- added joint Limb7_Limb8: type revolute, parent Limb7, child Limb8, origin xyz=0 2.4 0 rpy=0 0 0, axis 1 0 0, limit lower=-3.14159 upper=3.14159 effort=0.0 velocity=0.0
- added joint Limb8_Limb9: type revolute, parent Limb8, child Limb9, origin xyz=0 1.8 0 rpy=0 0 0, axis 1 0 0, limit lower=-3.14159 upper=3.14159 effort=0.0 velocity=0.0
- added joint Limb9_Limb10: type revolute, parent Limb9, child Limb10, origin xyz=0 1.6 0 rpy=0 0 0, axis 1 0 0, limit lower=-3.14159 upper=3.14159 effort=0.0 velocity=0.0
- joint Limb0_Limb1: origin xyz=0 0.375 0 rpy=0 0 0 -> xyz=0 0.525 0 rpy=0 0 0
- joint Limb1_Limb2: origin xyz=0 2.4 0 rpy=0 0 0 -> xyz=0 2.6 0 rpy=0 0 0
- joint Limb2_Limb3: origin xyz=0 2.5 0 rpy=0 0 0 -> xyz=0 1.9 0 rpy=0 0 0
- joint Limb3_Limb4: origin xyz=0 2.6 0 rpy=0 0 0 -> xyz=0 2.0 0 rpy=0 0 0
- joint Limb4_Limb5: origin xyz=0 2.7 0 rpy=0 0 0 -> xyz=0 2.9 0 rpy=0 0 0
- joint Limb5_Limb6: origin xyz=0 2.4 0 rpy=0 0 0 -> xyz=0 1.5 0 rpy=0 0 0
- joint Limb6_Limb7: origin xyz=0 2.1 0 rpy=0 0 0 -> xyz=0 2.8 0 rpy=0 0 0

Commit message: assign 6 README

File: body.urdf (robot description, URDF)
Before this commit: robot robot, 13 links, 12 joints
Links:
- removed link Limb10
- removed link Limb11
- removed link Limb12
- removed link Limb8
- removed link Limb9
- link Limb0: geometry collision box size=2.9 2.3 2.2; visual box size=2.9 2.3 2.2
- link Limb1: geometry collision box size=2.1 2.2 1.7; visual box size=2.1 2.2 1.7
- link Limb2: geometry collision box size=2.9 2.4 1.5; visual box size=2.9 2.4 1.5
- link Limb3: geometry collision box size=1.6 2.1 1.9; visual box size=1.6 2.1 1.9
- link Limb4: geometry collision box size=2.8 2.5 2.3; visual box size=2.8 2.5 2.3
- link Limb5: geometry collision box size=1.8 1.5 2.6; visual box size=1.8 1.5 2.6
- link Limb6: geometry collision box size=1.7 2.0 1.7; visual box size=1.7 2.0 1.7
- link Limb7: geometry collision box size=1.7 2.4 1.7; visual box size=1.7 2.4 1.7
Joints:
- removed joint Limb10_Limb11
- removed joint Limb11_Limb12
- removed joint Limb7_Limb8
- removed joint Limb8_Limb9
- removed joint Limb9_Limb10
- joint Limb0_Limb1: origin xyz=0 0.525 0 rpy=0 0 0 -> xyz=0 0.65 0 rpy=0 0 0
- joint Limb1_Limb2: origin xyz=0 2.6 0 rpy=0 0 0 -> xyz=0 2.2 0 rpy=0 0 0
- joint Limb2_Limb3: origin xyz=0 1.9 0 rpy=0 0 0 -> xyz=0 2.4 0 rpy=0 0 0
- joint Limb3_Limb4: origin xyz=0 2.0 0 rpy=0 0 0 -> xyz=0 2.1 0 rpy=0 0 0
- joint Limb4_Limb5: origin xyz=0 2.9 0 rpy=0 0 0 -> xyz=0 2.5 0 rpy=0 0 0
- joint Limb6_Limb7: origin xyz=0 2.8 0 rpy=0 0 0 -> xyz=0 2.0 0 rpy=0 0 0

Commit message: modifications on assign6

File: body.urdf (robot description, URDF)
Before this commit: robot robot, 8 links, 7 joints
Links:
- link Limb0: geometry collision box size=1.5 2.7 2.9; visual box size=1.5 2.7 2.9
- link Limb1: geometry collision box size=2.6 2.0 1.9; visual box size=2.6 2.0 1.9
- link Limb2: geometry collision box size=2.9 2.2 2.5; visual box size=2.9 2.2 2.5
- link Limb3: geometry collision box size=2.3 2.4 1.6; visual box size=2.3 2.4 1.6
- link Limb4: geometry collision box size=2.5 2.9 1.7; visual box size=2.5 2.9 1.7
- link Limb5: geometry collision box size=1.8 2.8 2.9; visual box size=1.8 2.8 2.9
- link Limb6: geometry collision box size=2.8 2.4 2.0; visual box size=2.8 2.4 2.0
- link Limb7: geometry collision box size=2.8 2.2 2.0; visual box size=2.8 2.2 2.0
Joints:
- joint Limb0_Limb1: origin xyz=0 0.65 0 rpy=0 0 0 -> xyz=0 1.35 0 rpy=0 0 0
- joint Limb1_Limb2: origin xyz=0 2.2 0 rpy=0 0 0 -> xyz=0 2.0 0 rpy=0 0 0
- joint Limb2_Limb3: origin xyz=0 2.4 0 rpy=0 0 0 -> xyz=0 2.2 0 rpy=0 0 0
- joint Limb3_Limb4: origin xyz=0 2.1 0 rpy=0 0 0 -> xyz=0 2.4 0 rpy=0 0 0
- joint Limb4_Limb5: origin xyz=0 2.5 0 rpy=0 0 0 -> xyz=0 2.9 0 rpy=0 0 0
- joint Limb5_Limb6: origin xyz=0 1.5 0 rpy=0 0 0 -> xyz=0 2.8 0 rpy=0 0 0
- joint Limb6_Limb7: origin xyz=0 2.0 0 rpy=0 0 0 -> xyz=0 2.4 0 rpy=0 0 0

Commit message: Finish assign7

File: body.urdf (robot description, URDF)
Before this commit: robot robot, 8 links, 7 joints
Links:
- added link Limb10, mass 1; collision box size=2.3 2.6 2.4; visual box size=2.3 2.6 2.4
- added link Limb11, mass 1; collision box size=1.2 2.6 2.4; visual box size=1.2 2.6 2.4
- added link Limb12, mass 1; collision box size=2.9 2.6 2.4; visual box size=2.9 2.6 2.4
- added link Limb13, mass 1; collision box size=2.0 2.6 2.4; visual box size=2.0 2.6 2.4
- added link Limb14, mass 1; collision box size=1.0 2.6 2.4; visual box size=1.0 2.6 2.4
- added link Limb15, mass 1; collision box size=1.5 2.6 2.4; visual box size=1.5 2.6 2.4
- added link Limb16, mass 1; collision box size=1.2 2.6 2.4; visual box size=1.2 2.6 2.4
- link Limb0: geometry collision box size=1.6 2.4 2.0; visual box size=1.6 2.4 2.0
- link Limb1: geometry collision box size=2.7 1.8 2.0; visual box size=2.7 1.8 2.0
- link Limb2: geometry collision box size=2.3 2.0 2.0; visual box size=2.3 2.0 2.0
- link Limb3: geometry collision box size=2.3 2.0 2.0; visual box size=2.3 2.0 2.0
- link Limb4: geometry collision box size=2.5 1.3 2.0; visual box size=2.5 1.3 2.0
- link Limb5: geometry collision box size=2.0 2.4 2.0; visual box size=2.0 2.4 2.0
- link Limb6: geometry collision box size=1.8 1.3 2.0; visual box size=1.8 1.3 2.0
- link Limb7: geometry collision box size=2.1 2.6 2.4; visual box size=2.1 2.6 2.4
Joints:
- added joint Limb10_Limb11: type revolute, parent Limb10, child Limb11, origin xyz=2.3 0 0 rpy=0 0 0, axis 0 1 0, limit lower=-3.14159 upper=3.14159 effort=0.0 velocity=0.0
- added joint Limb11_Limb12: type revolute, parent Limb11, child Limb12, origin xyz=1.2 0 0 rpy=0 0 0, axis 0 1 0, limit lower=-3.14159 upper=3.14159 effort=0.0 velocity=0.0
- added joint Limb12_Limb13: type revolute, parent Limb12, child Limb13, origin xyz=2.9 0 0 rpy=0 0 0, axis 0 1 0, limit lower=-3.14159 upper=3.14159 effort=0.0 velocity=0.0
- added joint Limb13_Limb14: type revolute, parent Limb13, child Limb14, origin xyz=2.0 0 0 rpy=0 0 0, axis 0 1 0, limit lower=-3.14159 upper=3.14159 effort=0.0 velocity=0.0
- added joint Limb14_Limb15: type revolute, parent Limb14, child Limb15, origin xyz=1.0 0 0 rpy=0 0 0, axis 0 1 0, limit lower=-3.14159 upper=3.14159 effort=0.0 velocity=0.0
- added joint Limb3_Limb10: type revolute, parent Limb3, child Limb10, origin xyz=1.15 0 0 rpy=0 0 0, axis 0 1 0, limit lower=-3.14159 upper=3.14159 effort=0.0 velocity=0.0
- added joint Limb5_Limb16: type revolute, parent Limb5, child Limb16, origin xyz=-1.0 0 0 rpy=0 0 0, axis 0 1 0, limit lower=-3.14159 upper=3.14159 effort=0.0 velocity=0.0
- joint Limb0_Limb1: origin xyz=0 1.35 0 rpy=0 0 0 -> xyz=0 1.2 0 rpy=0 0 0
- joint Limb1_Limb2: origin xyz=0 2.0 0 rpy=0 0 0 -> xyz=0 1.8 0 rpy=0 0 0
- joint Limb2_Limb3: origin xyz=0 2.2 0 rpy=0 0 0 -> xyz=0 2.0 0 rpy=0 0 0
- joint Limb3_Limb4: origin xyz=0 2.4 0 rpy=0 0 0 -> xyz=0 2.0 0 rpy=0 0 0
- joint Limb4_Limb5: origin xyz=0 2.9 0 rpy=0 0 0 -> xyz=0 1.3 0 rpy=0 0 0
- joint Limb5_Limb6: origin xyz=0 2.8 0 rpy=0 0 0 -> xyz=0 2.4 0 rpy=0 0 0
- joint Limb6_Limb7: origin xyz=0 2.4 0 rpy=0 0 0 -> xyz=0 1.3 0 rpy=0 0 0

Commit message: assign7 comment adds to solution.py

File: body.urdf (robot description, URDF)
Before this commit: robot robot, 15 links, 14 joints
Links:
- removed link Limb13
- removed link Limb14
- removed link Limb15
- removed link Limb16
- removed link Limb4
- removed link Limb5
- added link Limb8, mass 1; collision box size=1.5 2.2 1.5; visual box size=1.5 2.2 1.5
- added link Limb9, mass 1; collision box size=1.7 2.2 1.5; visual box size=1.7 2.2 1.5
- link Limb0: geometry collision box size=2.1 1.5 2.8; visual box size=2.1 1.5 2.8
- link Limb1: geometry collision box size=2.4 1.8 2.8; visual box size=2.4 1.8 2.8
- link Limb10: geometry collision box size=1.5 2.2 1.5; visual box size=1.5 2.2 1.5
- link Limb11: geometry collision box size=1.5 2.2 1.5; visual box size=1.5 2.2 1.5
- link Limb12: geometry collision box size=2.2 2.2 1.5; visual box size=2.2 2.2 1.5
- link Limb2: geometry collision box size=2.6 2.7 2.8; visual box size=2.6 2.7 2.8
- link Limb3: geometry collision box size=2.3 2.9 1.5; visual box size=2.3 2.9 1.5
- link Limb6: geometry collision box size=2.7 2.2 1.5; visual box size=2.7 2.2 1.5
- link Limb7: geometry collision box size=2.8 2.2 1.5; visual box size=2.8 2.2 1.5
Joints:
- removed joint Limb10_Limb11
- removed joint Limb11_Limb12
- removed joint Limb12_Limb13
- removed joint Limb13_Limb14
- removed joint Limb14_Limb15
- removed joint Limb3_Limb10
- removed joint Limb3_Limb4
- removed joint Limb4_Limb5
- removed joint Limb5_Limb16
- removed joint Limb5_Limb6
- removed joint Limb6_Limb7
- added joint Limb2_Limb10: type revolute, parent Limb2, child Limb10, origin xyz=-1.3 0 0 rpy=0 0 0, axis 0 1 0, limit lower=-3.14159 upper=3.14159 effort=0.0 velocity=0.0
- added joint Limb2_Limb7: type revolute, parent Limb2, child Limb7, origin xyz=1.3 0 0 rpy=0 0 0, axis 0 1 0, limit lower=-3.14159 upper=3.14159 effort=0.0 velocity=0.0
- added joint Limb3_Limb11: type revolute, parent Limb3, child Limb11, origin xyz=1.15 0 0 rpy=0 0 0, axis 0 1 0, limit lower=-3.14159 upper=3.14159 effort=0.0 velocity=0.0
- added joint Limb3_Limb12: type revolute, parent Limb3, child Limb12, origin xyz=1.15 0 0 rpy=0 0 0, axis 0 1 0, limit lower=-3.14159 upper=3.14159 effort=0.0 velocity=0.0
- added joint Limb3_Limb6: type revolute, parent Limb3, child Limb6, origin xyz=-1.15 0 0 rpy=0 0 0, axis 0 1 0, limit lower=-3.14159 upper=3.14159 effort=0.0 velocity=0.0
- added joint Limb7_Limb8: type revolute, parent Limb7, child Limb8, origin xyz=2.8 0 0 rpy=0 0 0, axis 0 1 0, limit lower=-3.14159 upper=3.14159 effort=0.0 velocity=0.0
- added joint Limb8_Limb9: type revolute, parent Limb8, child Limb9, origin xyz=1.5 0 0 rpy=0 0 0, axis 0 1 0, limit lower=-3.14159 upper=3.14159 effort=0.0 velocity=0.0
- joint Limb0_Limb1: origin xyz=0 1.2 0 rpy=0 0 0 -> xyz=0 0.75 0 rpy=0 0 0
- joint Limb2_Limb3: origin xyz=0 2.0 0 rpy=0 0 0 -> xyz=0 2.7 0 rpy=0 0 0

Commit message: added run.py moving to assign8

File: body.urdf (robot description, URDF)
Before this commit: robot robot, 11 links, 10 joints
Links:
- removed link Limb11
- removed link Limb12
- removed link Limb6
- removed link Limb7
- added link Limb4, mass 1; collision box size=2.3 1.0 2.5; visual box size=2.3 1.0 2.5
- added link Limb5, mass 1; collision box size=1.4 2.9 2.5; visual box size=1.4 2.9 2.5
- link Limb0: geometry collision box size=1.7 2.7 2.5; visual box size=1.7 2.7 2.5
- link Limb1: geometry collision box size=3.0 2.4 2.5; visual box size=3.0 2.4 2.5
- link Limb10: geometry collision box size=2.3 1.9 2.5; visual box size=2.3 1.9 2.5
- link Limb2: geometry collision box size=2.2 1.2 2.5; visual box size=2.2 1.2 2.5
- link Limb3: geometry collision box size=2.6 2.6 2.5; visual box size=2.6 2.6 2.5
- link Limb8: geometry collision box size=2.8 1.9 2.5; visual box size=2.8 1.9 2.5
- link Limb9: geometry collision box size=1.4 1.9 2.5; visual box size=1.4 1.9 2.5
Joints:
- removed joint Limb2_Limb10
- removed joint Limb2_Limb7
- removed joint Limb3_Limb11
- removed joint Limb3_Limb12
- removed joint Limb3_Limb6
- removed joint Limb7_Limb8
- removed joint Limb8_Limb9
- added joint Limb2_Limb8: type revolute, parent Limb2, child Limb8, origin xyz=1.1 0 0 rpy=0 0 0, axis 0 1 0, limit lower=-3.14159 upper=3.14159 effort=0.0 velocity=0.0
- added joint Limb3_Limb4: type revolute, parent Limb3, child Limb4, origin xyz=0 2.6 0 rpy=0 0 0, axis 1 0 0, limit lower=-3.14159 upper=3.14159 effort=0.0 velocity=0.0
- added joint Limb4_Limb5: type revolute, parent Limb4, child Limb5, origin xyz=0 1.0 0 rpy=0 0 0, axis 1 0 0, limit lower=-3.14159 upper=3.14159 effort=0.0 velocity=0.0
- added joint Limb4_Limb9: type revolute, parent Limb4, child Limb9, origin xyz=1.15 0 0 rpy=0 0 0, axis 0 1 0, limit lower=-3.14159 upper=3.14159 effort=0.0 velocity=0.0
- added joint Limb5_Limb10: type revolute, parent Limb5, child Limb10, origin xyz=0.7 0 0 rpy=0 0 0, axis 0 1 0, limit lower=-3.14159 upper=3.14159 effort=0.0 velocity=0.0
- joint Limb0_Limb1: origin xyz=0 0.75 0 rpy=0 0 0 -> xyz=0 1.35 0 rpy=0 0 0
- joint Limb1_Limb2: origin xyz=0 1.8 0 rpy=0 0 0 -> xyz=0 2.4 0 rpy=0 0 0
- joint Limb2_Limb3: origin xyz=0 2.7 0 rpy=0 0 0 -> xyz=0 1.2 0 rpy=0 0 0

Commit message: PHC working

File: body.urdf (robot description, URDF)
Before this commit: robot robot, 9 links, 8 joints
Links:
- removed link Limb4
- removed link Limb5
- added link Limb11, mass 1; collision box size=2.1 1.6 2.1; visual box size=2.1 1.6 2.1
- added link Limb12, mass 1; collision box size=1.9 1.6 2.1; visual box size=1.9 1.6 2.1
- added link Limb6, mass 1; collision box size=2.3 1.6 2.1; visual box size=2.3 1.6 2.1
- added link Limb7, mass 1; collision box size=2.2 1.6 2.1; visual box size=2.2 1.6 2.1
- link Limb0: geometry collision box size=1.4 2.2 2.9; visual box size=1.4 2.2 2.9
- link Limb1: geometry collision box size=1.1 1.9 2.9; visual box size=1.1 1.9 2.9
- link Limb10: geometry collision box size=1.8 1.6 2.1; visual box size=1.8 1.6 2.1
- link Limb2: geometry collision box size=2.5 1.7 2.9; visual box size=2.5 1.7 2.9
- link Limb3: geometry collision box size=1.6 1.0 2.1; visual box size=1.6 1.0 2.1
- link Limb8: geometry collision box size=2.0 1.6 2.1; visual box size=2.0 1.6 2.1
- link Limb9: geometry collision box size=1.0 1.6 2.1; visual box size=1.0 1.6 2.1
Joints:
- removed joint Limb3_Limb4
- removed joint Limb4_Limb5
- removed joint Limb4_Limb9
- removed joint Limb5_Limb10
- added joint Limb2_Limb10: type revolute, parent Limb2, child Limb10, origin xyz=-1.25 0 0 rpy=0 0 0, axis 0 1 0, limit lower=-3.14159 upper=3.14159 effort=0.0 velocity=0.0
- added joint Limb2_Limb11: type revolute, parent Limb2, child Limb11, origin xyz=1.25 0 0 rpy=0 0 0, axis 0 1 0, limit lower=-3.14159 upper=3.14159 effort=0.0 velocity=0.0
- added joint Limb2_Limb6: type revolute, parent Limb2, child Limb6, origin xyz=1.25 0 0 rpy=0 0 0, axis 0 1 0, limit lower=-3.14159 upper=3.14159 effort=0.0 velocity=0.0
- added joint Limb3_Limb12: type revolute, parent Limb3, child Limb12, origin xyz=-0.8 0 0 rpy=0 0 0, axis 0 1 0, limit lower=-3.14159 upper=3.14159 effort=0.0 velocity=0.0
- added joint Limb3_Limb7: type revolute, parent Limb3, child Limb7, origin xyz=-0.8 0 0 rpy=0 0 0, axis 0 1 0, limit lower=-3.14159 upper=3.14159 effort=0.0 velocity=0.0
- added joint Limb3_Limb9: type revolute, parent Limb3, child Limb9, origin xyz=-0.8 0 0 rpy=0 0 0, axis 0 1 0, limit lower=-3.14159 upper=3.14159 effort=0.0 velocity=0.0
- joint Limb0_Limb1: origin xyz=0 1.35 0 rpy=0 0 0 -> xyz=0 1.1 0 rpy=0 0 0
- joint Limb1_Limb2: origin xyz=0 2.4 0 rpy=0 0 0 -> xyz=0 1.9 0 rpy=0 0 0
- joint Limb2_Limb3: origin xyz=0 1.2 0 rpy=0 0 0 -> xyz=0 1.7 0 rpy=0 0 0
- joint Limb2_Limb8: origin xyz=1.1 0 0 rpy=0 0 0 -> xyz=1.25 0 0 rpy=0 0 0
