Commit message: close with assign8

File: body.urdf (robot description, URDF)
Before this commit: robot robot, 11 links, 10 joints
Links:
- removed link Limb10
- removed link Limb11
- removed link Limb12
- removed link Limb3
- removed link Limb6
- removed link Limb7
- removed link Limb8
- removed link Limb9
- added link BotLimb0, mass 1; collision box size=1.4 0.7 1.1; visual box size=1.4 0.7 1.1
- added link BotLimb1, mass 1; collision box size=0.7 0.7 1.4; visual box size=0.7 0.7 1.4
- link Limb0: geometry collision box size=1.4 0.7 1.1; visual box size=1.4 0.7 1.1
- link Limb1: geometry collision box size=0.7 0.7 1.4; visual box size=0.7 0.7 1.4
- link Limb2: geometry collision box size=1.4 0.7 1.1; visual box size=1.4 0.7 1.1
Joints:
- removed joint Limb0_Limb1
- removed joint Limb1_Limb2
- removed joint Limb2_Limb10
- removed joint Limb2_Limb11
- removed joint Limb2_Limb3
- removed joint Limb2_Limb6
- removed joint Limb2_Limb8
- removed joint Limb3_Limb12
- removed joint Limb3_Limb7
- removed joint Limb3_Limb9
- added joint BotLimb0_Limb1: type revolute, parent BotLimb0, child Limb1, origin xyz=0 0.7 0 rpy=0 0 0, axis 1 0 0, limit lower=-3.14159 upper=3.14159 effort=0.0 velocity=0.0
- added joint BotLimb1_Limb2: type revolute, parent BotLimb1, child Limb2, origin xyz=0 0.7 0 rpy=0 0 0, axis 1 0 0, limit lower=-3.14159 upper=3.14159 effort=0.0 velocity=0.0
- added joint Limb0_BotLimb0: type revolute, parent Limb0, child BotLimb0, origin xyz=0 0.35 1.1 rpy=0 0 0, axis 1 0 0, limit lower=-3.14159 upper=3.14159 effort=0.0 velocity=0.0
- added joint Limb1_BotLimb1: type revolute, parent Limb1, child BotLimb1, origin xyz=0 0.7 0 rpy=0 0 0, axis 1 0 0, limit lower=-3.14159 upper=3.14159 effort=0.0 velocity=0.0

Commit message: Finished assign 8

File: body.urdf (robot description, URDF)
Before this commit: robot robot, 5 links, 4 joints
Links:
- added link BotLimb2, mass 1; collision box size=1.1 1.1 1.1; visual box size=1.1 1.1 1.1
- added link BotLimb3, mass 1; collision box size=0.8 1.0 1.1; visual box size=0.8 1.0 1.1
- added link Limb3, mass 1; collision box size=0.8 1.0 1.1; visual box size=0.8 1.0 1.1
- added link Limb4, mass 1; collision box size=1.6 1.0 0.9; visual box size=1.6 1.0 0.9
- added link Limb7, mass 1; collision box size=0.9 1.8 1.7; visual box size=0.9 1.8 1.7
- added link Limb9, mass 1; collision box size=2.1 1.8 1.7; visual box size=2.1 1.8 1.7
- link BotLimb0: geometry collision box size=1.6 1.0 0.9; visual box size=1.6 1.0 0.9
- link BotLimb1: geometry collision box size=1.0 0.8 2.1; visual box size=1.0 0.8 2.1
- link Limb0: geometry collision box size=1.6 1.0 0.9; visual box size=1.6 1.0 0.9
- link Limb1: geometry collision box size=1.0 0.8 2.1; visual box size=1.0 0.8 2.1
- link Limb2: geometry collision box size=1.1 1.1 1.1; visual box size=1.1 1.1 1.1
Joints:
- added joint BotLimb2_Limb3: type revolute, parent BotLimb2, child Limb3, origin xyz=0 1.1 0 rpy=0 0 0, axis 1 0 0, limit lower=-3.14159 upper=3.14159 effort=0.0 velocity=0.0
- added joint BotLimb3_Limb4: type revolute, parent BotLimb3, child Limb4, origin xyz=0 1.0 0 rpy=0 0 0, axis 1 0 0, limit lower=-3.14159 upper=3.14159 effort=0.0 velocity=0.0
- added joint Limb2_BotLimb2: type revolute, parent Limb2, child BotLimb2, origin xyz=0 1.1 0 rpy=0 0 0, axis 1 0 0, limit lower=-3.14159 upper=3.14159 effort=0.0 velocity=0.0
- added joint Limb2_Limb9: type revolute, parent Limb2, child Limb9, origin xyz=-0.55 0 -0.55 rpy=0 0 0, axis 0 1 1, limit lower=-3.14159 upper=3.14159 effort=0.0 velocity=0.0
- added joint Limb3_BotLimb3: type revolute, parent Limb3, child BotLimb3, origin xyz=0 1.0 0 rpy=0 0 0, axis 1 0 0, limit lower=-3.14159 upper=3.14159 effort=0.0 velocity=0.0
- added joint Limb4_Limb7: type revolute, parent Limb4, child Limb7, origin xyz=0.45 0 -0.9 rpy=0 0 0, axis 0 1 0, limit lower=-3.14159 upper=3.14159 effort=0.0 velocity=0.0
- joint BotLimb0_Limb1: origin xyz=0 0.7 0 rpy=0 0 0 -> xyz=0 1.0 0 rpy=0 0 0
- joint BotLimb1_Limb2: origin xyz=0 0.7 0 rpy=0 0 0 -> xyz=0 0.8 0 rpy=0 0 0
- joint Limb0_BotLimb0: origin xyz=0 0.35 1.1 rpy=0 0 0 -> xyz=0 0.5 0.9 rpy=0 0 0
- joint Limb1_BotLimb1: origin xyz=0 0.7 0 rpy=0 0 0 -> xyz=0 0.8 0 rpy=0 0 0

Commit message: 5 graphs done

File: body.urdf (robot description, URDF)
Before this commit: robot robot, 11 links, 10 joints
Links:
- removed link Limb7
- added link BotLimb4, mass 1; collision box size=1.8 0.9 1.7; visual box size=1.8 0.9 1.7
- added link Limb10, mass 1; collision box size=1.3 2.3 2.5; visual box size=1.3 2.3 2.5
- added link Limb11, mass 1; collision box size=1.0 2.3 2.5; visual box size=1.0 2.3 2.5
- added link Limb13, mass 1; collision box size=1.6 2.3 2.5; visual box size=1.6 2.3 2.5
- added link Limb5, mass 1; collision box size=1.4 1.6 1.7; visual box size=1.4 1.6 1.7
- added link Limb8, mass 1; collision box size=0.8 2.3 2.5; visual box size=0.8 2.3 2.5
- link BotLimb0: geometry collision box size=1.4 1.6 1.7; visual box size=1.4 1.6 1.7
- link BotLimb1: geometry collision box size=1.2 1.4 1.1; visual box size=1.2 1.4 1.1
- link BotLimb2: geometry collision box size=1.2 2.0 2.1; visual box size=1.2 2.0 2.1
- link BotLimb3: geometry collision box size=0.8 1.5 1.4; visual box size=0.8 1.5 1.4
- link Limb0: geometry collision box size=1.4 1.6 1.7; visual box size=1.4 1.6 1.7
- link Limb1: geometry collision box size=1.2 1.4 1.1; visual box size=1.2 1.4 1.1
- link Limb2: geometry collision box size=1.2 2.0 2.1; visual box size=1.2 2.0 2.1
- link Limb3: geometry collision box size=0.8 1.5 1.4; visual box size=0.8 1.5 1.4
- link Limb4: geometry collision box size=1.8 0.9 1.7; visual box size=1.8 0.9 1.7
- link Limb9: geometry collision box size=0.9 2.3 2.5; visual box size=0.9 2.3 2.5
Joints:
- removed joint Limb4_Limb7
- added joint BotLimb4_Limb5: type revolute, parent BotLimb4, child Limb5, origin xyz=0 0.9 0 rpy=0 0 0, axis 1 0 0, limit lower=-3.14159 upper=3.14159 effort=0.0 velocity=0.0
- added joint Limb3_Limb10: type revolute, parent Limb3, child Limb10, origin xyz=-0.4 0 -0.75 rpy=0 0 0, axis 0 1 0, limit lower=-3.14159 upper=3.14159 effort=0.0 velocity=0.0
- added joint Limb3_Limb13: type revolute, parent Limb3, child Limb13, origin xyz=0.4 0 -0.75 rpy=0 0 0, axis 0 1 0, limit lower=-3.14159 upper=3.14159 effort=0.0 velocity=0.0
- added joint Limb4_BotLimb4: type revolute, parent Limb4, child BotLimb4, origin xyz=0 0.9 0 rpy=0 0 0, axis 1 0 0, limit lower=-3.14159 upper=3.14159 effort=0.0 velocity=0.0
- added joint Limb4_Limb11: type revolute, parent Limb4, child Limb11, origin xyz=0.9 0 -0.45 rpy=0 0 0, axis 0 1 0, limit lower=-3.14159 upper=3.14159 effort=0.0 velocity=0.0
- added joint Limb5_Limb8: type revolute, parent Limb5, child Limb8, origin xyz=0.85 0 -0.55 rpy=0 0 0, axis 0 1 0, limit lower=-3.14159 upper=3.14159 effort=0.0 velocity=0.0
- joint BotLimb0_Limb1: origin xyz=0 1.0 0 rpy=0 0 0 -> xyz=0 1.6 0 rpy=0 0 0
- joint BotLimb1_Limb2: origin xyz=0 0.8 0 rpy=0 0 0 -> xyz=0 1.4 0 rpy=0 0 0
- joint BotLimb2_Limb3: origin xyz=0 1.1 0 rpy=0 0 0 -> xyz=0 2.0 0 rpy=0 0 0
- joint BotLimb3_Limb4: origin xyz=0 1.0 0 rpy=0 0 0 -> xyz=0 1.5 0 rpy=0 0 0
- joint Limb0_BotLimb0: origin xyz=0 0.5 0.9 rpy=0 0 0 -> xyz=0 0.8 2.7 rpy=0 0 0
- joint Limb1_BotLimb1: origin xyz=0 0.8 0 rpy=0 0 0 -> xyz=0 1.4 0 rpy=0 0 0
- joint Limb2_BotLimb2: origin xyz=0 1.1 0 rpy=0 0 0 -> xyz=0 2.0 0 rpy=0 0 0
- joint Limb2_Limb9: axis 0 1 1 -> 0 1 0; origin xyz=-0.55 0 -0.55 rpy=0 0 0 -> xyz=0.6 0 -1.0 rpy=0 0 0
- joint Limb3_BotLimb3: origin xyz=0 1.0 0 rpy=0 0 0 -> xyz=0 1.5 0 rpy=0 0 0

Commit message: video

File: body.urdf (robot description, URDF)
Before this commit: robot robot, 16 links, 15 joints
Links:
- removed link Limb13
- added link Limb14, mass 1; collision box size=0.8 2.3 1.5; visual box size=0.8 2.3 1.5
- added link Limb17, mass 1; collision box size=1.9 2.3 1.5; visual box size=1.9 2.3 1.5
- link BotLimb0: geometry collision box size=1.7 1.3 1.7; visual box size=1.7 1.3 1.7
- link BotLimb1: geometry collision box size=1.1 0.8 1.4; visual box size=1.1 0.8 1.4
- link BotLimb2: geometry collision box size=2.1 1.7 1.0; visual box size=2.1 1.7 1.0
- link BotLimb3: geometry collision box size=0.8 2.0 1.8; visual box size=0.8 2.0 1.8
- link BotLimb4: geometry collision box size=1.4 1.7 1.5; visual box size=1.4 1.7 1.5
- link Limb0: geometry collision box size=1.7 1.3 1.7; visual box size=1.7 1.3 1.7
- link Limb1: geometry collision box size=1.1 0.8 1.4; visual box size=1.1 0.8 1.4
- link Limb10: geometry collision box size=1.4 2.3 1.5; visual box size=1.4 2.3 1.5
- link Limb11: geometry collision box size=2.0 2.3 1.5; visual box size=2.0 2.3 1.5
- link Limb2: geometry collision box size=2.1 1.7 1.0; visual box size=2.1 1.7 1.0
- link Limb3: geometry collision box size=0.8 2.0 1.8; visual box size=0.8 2.0 1.8
- link Limb4: geometry collision box size=1.4 1.7 1.5; visual box size=1.4 1.7 1.5
- link Limb5: geometry collision box size=1.7 1.3 1.7; visual box size=1.7 1.3 1.7
- link Limb8: geometry collision box size=1.8 2.3 1.5; visual box size=1.8 2.3 1.5
- link Limb9: geometry collision box size=0.9 2.3 1.5; visual box size=0.9 2.3 1.5
Joints:
- removed joint Limb2_Limb9
- removed joint Limb3_Limb10
- removed joint Limb3_Limb13
- removed joint Limb4_Limb11
- removed joint Limb5_Limb8
- added joint Limb2_Limb10: type revolute, parent Limb2, child Limb10, origin xyz=-1.05 0 -0.85 rpy=0 0 0, axis 0 1 0, limit lower=-3.14159 upper=3.14159 effort=0.0 velocity=0.0
- added joint Limb2_Limb14: type revolute, parent Limb2, child Limb14, origin xyz=1.05 0 -0.85 rpy=0 0 0, axis 0 1 0, limit lower=-3.14159 upper=3.14159 effort=0.0 velocity=0.0
- added joint Limb2_Limb8: type revolute, parent Limb2, child Limb8, origin xyz=-1.05 0 -0.85 rpy=0 0 0, axis 0 1 0, limit lower=-3.14159 upper=3.14159 effort=0.0 velocity=0.0
- added joint Limb3_Limb9: type revolute, parent Limb3, child Limb9, origin xyz=0.4 0 -1.0 rpy=0 0 0, axis 0 1 0, limit lower=-3.14159 upper=3.14159 effort=0.0 velocity=0.0
- added joint Limb4_Limb17: type revolute, parent Limb4, child Limb17, origin xyz=0.7 0 -0.85 rpy=0 0 0, axis 0 1 0, limit lower=-3.14159 upper=3.14159 effort=0.0 velocity=0.0
- added joint Limb5_Limb11: type revolute, parent Limb5, child Limb11, origin xyz=-0.9 0 -0.75 rpy=0 0 0, axis 0 1 0, limit lower=-3.14159 upper=3.14159 effort=0.0 velocity=0.0
- joint BotLimb0_Limb1: origin xyz=0 1.6 0 rpy=0 0 0 -> xyz=0 1.3 0 rpy=0 0 0
- joint BotLimb1_Limb2: origin xyz=0 1.4 0 rpy=0 0 0 -> xyz=0 0.8 0 rpy=0 0 0
- joint BotLimb2_Limb3: origin xyz=0 2.0 0 rpy=0 0 0 -> xyz=0 1.7 0 rpy=0 0 0
- joint BotLimb3_Limb4: origin xyz=0 1.5 0 rpy=0 0 0 -> xyz=0 2.0 0 rpy=0 0 0
- joint BotLimb4_Limb5: origin xyz=0 0.9 0 rpy=0 0 0 -> xyz=0 1.7 0 rpy=0 0 0
- joint Limb0_BotLimb0: origin xyz=0 0.8 2.7 rpy=0 0 0 -> xyz=0 0.65 2.7 rpy=0 0 0
- joint Limb1_BotLimb1: origin xyz=0 1.4 0 rpy=0 0 0 -> xyz=0 0.8 0 rpy=0 0 0
- joint Limb2_BotLimb2: origin xyz=0 2.0 0 rpy=0 0 0 -> xyz=0 1.7 0 rpy=0 0 0
- joint Limb3_BotLimb3: origin xyz=0 1.5 0 rpy=0 0 0 -> xyz=0 2.0 0 rpy=0 0 0
- joint Limb4_BotLimb4: origin xyz=0 0.9 0 rpy=0 0 0 -> xyz=0 1.7 0 rpy=0 0 0

Commit message: added 2 figures

File: body.urdf (robot description, URDF)
Before this commit: robot robot, 17 links, 16 joints
Links:
- removed link Limb8
- added link BotLimb5, mass 1; collision box size=1.9 1.8 1.8; visual box size=1.9 1.8 1.8
- added link Limb12, mass 1; collision box size=2.2 2.4 2.4; visual box size=2.2 2.4 2.4
- added link Limb15, mass 1; collision box size=1.8 2.4 2.4; visual box size=1.8 2.4 2.4
- added link Limb16, mass 1; collision box size=1.1 2.4 2.4; visual box size=1.1 2.4 2.4
- added link Limb22, mass 1; collision box size=1.6 2.4 2.4; visual box size=1.6 2.4 2.4
- added link Limb6, mass 1; collision box size=1.3 1.4 2.1; visual box size=1.3 1.4 2.1
- link BotLimb0: geometry collision box size=1.3 1.4 2.1; visual box size=1.3 1.4 2.1
- link BotLimb1: geometry collision box size=1.1 1.0 2.2; visual box size=1.1 1.0 2.2
- link BotLimb2: geometry collision box size=1.7 1.2 1.2; visual box size=1.7 1.2 1.2
- link BotLimb3: geometry collision box size=1.8 1.1 1.5; visual box size=1.8 1.1 1.5
- link BotLimb4: geometry collision box size=1.7 1.4 2.0; visual box size=1.7 1.4 2.0
- link Limb0: geometry collision box size=1.3 1.4 2.1; visual box size=1.3 1.4 2.1
- link Limb1: geometry collision box size=1.1 1.0 2.2; visual box size=1.1 1.0 2.2
- link Limb10: geometry collision box size=0.8 2.4 2.4; visual box size=0.8 2.4 2.4
- link Limb11: geometry collision box size=2.2 2.4 2.4; visual box size=2.2 2.4 2.4
- link Limb14: geometry collision box size=2.2 2.4 2.4; visual box size=2.2 2.4 2.4
- link Limb17: geometry collision box size=1.4 2.4 2.4; visual box size=1.4 2.4 2.4
- link Limb2: geometry collision box size=1.7 1.2 1.2; visual box size=1.7 1.2 1.2
- link Limb3: geometry collision box size=1.8 1.1 1.5; visual box size=1.8 1.1 1.5
- link Limb4: geometry collision box size=1.7 1.4 2.0; visual box size=1.7 1.4 2.0
- link Limb5: geometry collision box size=1.9 1.8 1.8; visual box size=1.9 1.8 1.8
- link Limb9: geometry collision box size=1.6 2.4 2.4; visual box size=1.6 2.4 2.4
Joints:
- removed joint Limb2_Limb10
- removed joint Limb2_Limb14
- removed joint Limb2_Limb8
- removed joint Limb3_Limb9
- removed joint Limb4_Limb17
- added joint BotLimb5_Limb6: type revolute, parent BotLimb5, child Limb6, origin xyz=0 1.8 0 rpy=0 0 0, axis 1 0 0, limit lower=-3.14159 upper=3.14159 effort=0.0 velocity=0.0
- added joint Limb2_Limb12: type revolute, parent Limb2, child Limb12, origin xyz=0.85 0 -0.6 rpy=0 0 0, axis 0 1 0, limit lower=-3.14159 upper=3.14159 effort=0.0 velocity=0.0
- added joint Limb3_Limb10: type revolute, parent Limb3, child Limb10, origin xyz=0.9 0 -0.55 rpy=0 0 0, axis 0 1 0, limit lower=-3.14159 upper=3.14159 effort=0.0 velocity=0.0
- added joint Limb5_BotLimb5: type revolute, parent Limb5, child BotLimb5, origin xyz=0 1.8 0 rpy=0 0 0, axis 1 0 0, limit lower=-3.14159 upper=3.14159 effort=0.0 velocity=0.0
- added joint Limb5_Limb14: type revolute, parent Limb5, child Limb14, origin xyz=-0.95 0 -0.9 rpy=0 0 0, axis 0 1 0, limit lower=-3.14159 upper=3.14159 effort=0.0 velocity=0.0
- added joint Limb5_Limb15: type revolute, parent Limb5, child Limb15, origin xyz=-0.95 0 -0.9 rpy=0 0 0, axis 0 1 0, limit lower=-3.14159 upper=3.14159 effort=0.0 velocity=0.0
- added joint Limb5_Limb17: type revolute, parent Limb5, child Limb17, origin xyz=-0.95 0 -0.9 rpy=0 0 0, axis 0 1 0, limit lower=-3.14159 upper=3.14159 effort=0.0 velocity=0.0
- added joint Limb5_Limb22: type revolute, parent Limb5, child Limb22, origin xyz=0.95 0 -0.9 rpy=0 0 0, axis 0 1 0, limit lower=-3.14159 upper=3.14159 effort=0.0 velocity=0.0
- added joint Limb6_Limb16: type revolute, parent Limb6, child Limb16, origin xyz=1.1 0 -1.0 rpy=0 0 0, axis 0 1 0, limit lower=-3.14159 upper=3.14159 effort=0.0 velocity=0.0
- added joint Limb6_Limb9: type revolute, parent Limb6, child Limb9, origin xyz=-1.1 0 -1.0 rpy=0 0 0, axis 0 1 0, limit lower=-3.14159 upper=3.14159 effort=0.0 velocity=0.0
- joint BotLimb0_Limb1: origin xyz=0 1.3 0 rpy=0 0 0 -> xyz=0 1.4 0 rpy=0 0 0
- joint BotLimb1_Limb2: origin xyz=0 0.8 0 rpy=0 0 0 -> xyz=0 1.0 0 rpy=0 0 0
- joint BotLimb2_Limb3: origin xyz=0 1.7 0 rpy=0 0 0 -> xyz=0 1.2 0 rpy=0 0 0
- joint BotLimb3_Limb4: origin xyz=0 2.0 0 rpy=0 0 0 -> xyz=0 1.1 0 rpy=0 0 0
- joint BotLimb4_Limb5: origin xyz=0 1.7 0 rpy=0 0 0 -> xyz=0 1.4 0 rpy=0 0 0
- joint Limb0_BotLimb0: origin xyz=0 0.65 2.7 rpy=0 0 0 -> xyz=0 0.7 3.1 rpy=0 0 0
- joint Limb1_BotLimb1: origin xyz=0 0.8 0 rpy=0 0 0 -> xyz=0 1.0 0 rpy=0 0 0
- joint Limb2_BotLimb2: origin xyz=0 1.7 0 rpy=0 0 0 -> xyz=0 1.2 0 rpy=0 0 0
- joint Limb3_BotLimb3: origin xyz=0 2.0 0 rpy=0 0 0 -> xyz=0 1.1 0 rpy=0 0 0
- joint Limb4_BotLimb4: origin xyz=0 1.7 0 rpy=0 0 0 -> xyz=0 1.4 0 rpy=0 0 0
- joint Limb5_Limb11: origin xyz=-0.9 0 -0.75 rpy=0 0 0 -> xyz=-0.95 0 -0.9 rpy=0 0 0

Commit message: BROLL Left

File: body.urdf (robot description, URDF)
Before this commit: robot robot, 22 links, 21 joints
Links:
- removed link Limb14
- removed link Limb17
- removed link Limb22
- added link Limb13, mass 1; collision box size=1.3 2.2 2.7; visual box size=1.3 2.2 2.7
- added link Limb18, mass 1; collision box size=0.9 2.2 2.7; visual box size=0.9 2.2 2.7
- link BotLimb0: geometry collision box size=1.0 1.9 2.1; visual box size=1.0 1.9 2.1
- link BotLimb1: geometry collision box size=1.9 1.5 1.7; visual box size=1.9 1.5 1.7
- link BotLimb2: geometry collision box size=1.0 1.6 1.9; visual box size=1.0 1.6 1.9
- link BotLimb3: geometry collision box size=0.9 1.0 1.6; visual box size=0.9 1.0 1.6
- link BotLimb4: geometry collision box size=1.1 1.1 1.9; visual box size=1.1 1.1 1.9
- link BotLimb5: geometry collision box size=1.2 1.7 2.0; visual box size=1.2 1.7 2.0
- link Limb0: geometry collision box size=1.0 1.9 2.1; visual box size=1.0 1.9 2.1
- link Limb1: geometry collision box size=1.9 1.5 1.7; visual box size=1.9 1.5 1.7
- link Limb10: geometry collision box size=2.1 2.2 2.7; visual box size=2.1 2.2 2.7
- link Limb11: geometry collision box size=1.6 2.2 2.7; visual box size=1.6 2.2 2.7
- link Limb12: geometry collision box size=1.1 2.2 2.7; visual box size=1.1 2.2 2.7
- link Limb15: geometry collision box size=0.8 2.2 2.7; visual box size=0.8 2.2 2.7
- link Limb16: geometry collision box size=1.6 2.2 2.7; visual box size=1.6 2.2 2.7
- link Limb2: geometry collision box size=1.0 1.6 1.9; visual box size=1.0 1.6 1.9
- link Limb3: geometry collision box size=0.9 1.0 1.6; visual box size=0.9 1.0 1.6
- link Limb4: geometry collision box size=1.1 1.1 1.9; visual box size=1.1 1.1 1.9
- link Limb5: geometry collision box size=1.2 1.7 2.0; visual box size=1.2 1.7 2.0
- link Limb6: geometry collision box size=1.0 1.9 2.1; visual box size=1.0 1.9 2.1
- link Limb9: geometry collision box size=1.8 2.2 2.7; visual box size=1.8 2.2 2.7
Joints:
- removed joint Limb2_Limb12
- removed joint Limb3_Limb10
- removed joint Limb5_Limb11
- removed joint Limb5_Limb14
- removed joint Limb5_Limb15
- removed joint Limb5_Limb17
- removed joint Limb5_Limb22
- removed joint Limb6_Limb16
- removed joint Limb6_Limb9
- added joint Limb3_Limb9: type revolute, parent Limb3, child Limb9, origin xyz=0.45 0 -0.5 rpy=0 0 0, axis 0 1 0, limit lower=-3.14159 upper=3.14159 effort=0.0 velocity=0.0
- added joint Limb4_Limb11: type revolute, parent Limb4, child Limb11, origin xyz=-0.55 0 -0.55 rpy=0 0 0, axis 0 1 0, limit lower=-3.14159 upper=3.14159 effort=0.0 velocity=0.0
- added joint Limb4_Limb12: type revolute, parent Limb4, child Limb12, origin xyz=0.55 0 -0.55 rpy=0 0 0, axis 0 1 0, limit lower=-3.14159 upper=3.14159 effort=0.0 velocity=0.0
- added joint Limb5_Limb10: type revolute, parent Limb5, child Limb10, origin xyz=-0.6 0 -0.85 rpy=0 0 0, axis 0 1 0, limit lower=-3.14159 upper=3.14159 effort=0.0 velocity=0.0
- added joint Limb5_Limb16: type revolute, parent Limb5, child Limb16, origin xyz=-0.6 0 -0.85 rpy=0 0 0, axis 0 1 0, limit lower=-3.14159 upper=3.14159 effort=0.0 velocity=0.0
- added joint Limb6_Limb13: type revolute, parent Limb6, child Limb13, origin xyz=-0.4 0 -0.5 rpy=0 0 0, axis 0 1 0, limit lower=-3.14159 upper=3.14159 effort=0.0 velocity=0.0
- added joint Limb6_Limb15: type revolute, parent Limb6, child Limb15, origin xyz=-0.4 0 -0.5 rpy=0 0 0, axis 0 1 0, limit lower=-3.14159 upper=3.14159 effort=0.0 velocity=0.0
- added joint Limb6_Limb18: type revolute, parent Limb6, child Limb18, origin xyz=0.4 0 -0.5 rpy=0 0 0, axis 0 1 0, limit lower=-3.14159 upper=3.14159 effort=0.0 velocity=0.0
- joint BotLimb0_Limb1: origin xyz=0 1.4 0 rpy=0 0 0 -> xyz=0 1.9 0 rpy=0 0 0
- joint BotLimb1_Limb2: origin xyz=0 1.0 0 rpy=0 0 0 -> xyz=0 1.5 0 rpy=0 0 0
- joint BotLimb2_Limb3: origin xyz=0 1.2 0 rpy=0 0 0 -> xyz=0 1.6 0 rpy=0 0 0
- joint BotLimb3_Limb4: origin xyz=0 1.1 0 rpy=0 0 0 -> xyz=0 1.0 0 rpy=0 0 0
- joint BotLimb4_Limb5: origin xyz=0 1.4 0 rpy=0 0 0 -> xyz=0 1.1 0 rpy=0 0 0
- joint BotLimb5_Limb6: origin xyz=0 1.8 0 rpy=0 0 0 -> xyz=0 1.7 0 rpy=0 0 0
- joint Limb0_BotLimb0: origin xyz=0 0.7 3.1 rpy=0 0 0 -> xyz=0 0.95 3.1 rpy=0 0 0
- joint Limb1_BotLimb1: origin xyz=0 1.0 0 rpy=0 0 0 -> xyz=0 1.5 0 rpy=0 0 0
- joint Limb2_BotLimb2: origin xyz=0 1.2 0 rpy=0 0 0 -> xyz=0 1.6 0 rpy=0 0 0
- joint Limb3_BotLimb3: origin xyz=0 1.1 0 rpy=0 0 0 -> xyz=0 1.0 0 rpy=0 0 0
- joint Limb4_BotLimb4: origin xyz=0 1.4 0 rpy=0 0 0 -> xyz=0 1.1 0 rpy=0 0 0
- joint Limb5_BotLimb5: origin xyz=0 1.8 0 rpy=0 0 0 -> xyz=0 1.7 0 rpy=0 0 0
