Commit message: BROLL Left

File: body.urdf (robot description, URDF)
Before this commit: robot robot, 21 links, 20 joints
Links:
- removed link Limb10
- removed link Limb16
- removed link Limb18
- removed link Limb9
- added link BotLimb6, mass 1; collision box size=1.0 1.4 1.1; visual box size=1.0 1.4 1.1
- added link BotLimb7, mass 1; collision box size=1.1 1.2 1.9; visual box size=1.1 1.2 1.9
- added link Limb14, mass 1; collision box size=1.0 2.0 1.9; visual box size=1.0 2.0 1.9
- added link Limb7, mass 1; collision box size=1.1 1.2 1.9; visual box size=1.1 1.2 1.9
- added link Limb8, mass 1; collision box size=1.9 2.1 1.7; visual box size=1.9 2.1 1.7
- link BotLimb0: geometry collision box size=1.9 2.1 1.7; visual box size=1.9 2.1 1.7
- link BotLimb1: geometry collision box size=1.6 1.3 1.8; visual box size=1.6 1.3 1.8
- link BotLimb2: geometry collision box size=1.2 1.5 2.1; visual box size=1.2 1.5 2.1
- link BotLimb3: geometry collision box size=2.2 0.8 2.0; visual box size=2.2 0.8 2.0
- link BotLimb4: geometry collision box size=1.5 1.2 1.9; visual box size=1.5 1.2 1.9
- link BotLimb5: geometry collision box size=1.8 2.1 2.1; visual box size=1.8 2.1 2.1
- link Limb0: geometry collision box size=1.9 2.1 1.7; visual box size=1.9 2.1 1.7
- link Limb1: geometry collision box size=1.6 1.3 1.8; visual box size=1.6 1.3 1.8
- link Limb11: geometry collision box size=1.6 2.0 1.9; visual box size=1.6 2.0 1.9
- link Limb12: geometry collision box size=1.9 2.0 1.9; visual box size=1.9 2.0 1.9
- link Limb13: geometry collision box size=1.4 2.0 1.9; visual box size=1.4 2.0 1.9
- link Limb15: geometry collision box size=1.0 2.0 1.9; visual box size=1.0 2.0 1.9
- link Limb2: geometry collision box size=1.2 1.5 2.1; visual box size=1.2 1.5 2.1
- link Limb3: geometry collision box size=2.2 0.8 2.0; visual box size=2.2 0.8 2.0
- link Limb4: geometry collision box size=1.5 1.2 1.9; visual box size=1.5 1.2 1.9
- link Limb5: geometry collision box size=1.8 2.1 2.1; visual box size=1.8 2.1 2.1
- link Limb6: geometry collision box size=1.0 1.4 1.1; visual box size=1.0 1.4 1.1
Joints:
- removed joint Limb3_Limb9
- removed joint Limb4_Limb11
- removed joint Limb4_Limb12
- removed joint Limb5_Limb10
- removed joint Limb5_Limb16
- removed joint Limb6_Limb13
- removed joint Limb6_Limb15
- removed joint Limb6_Limb18
- added joint BotLimb6_Limb7: type revolute, parent BotLimb6, child Limb7, origin xyz=0 1.4 0 rpy=0 0 0, axis 1 0 0, limit lower=-3.14159 upper=3.14159 effort=0.0 velocity=0.0
- added joint BotLimb7_Limb8: type revolute, parent BotLimb7, child Limb8, origin xyz=0 1.2 0 rpy=0 0 0, axis 1 0 0, limit lower=-3.14159 upper=3.14159 effort=0.0 velocity=0.0
- added joint Limb2_Limb11: type revolute, parent Limb2, child Limb11, origin xyz=-0.6 0 -0.75 rpy=0 0 0, axis 0 1 0, limit lower=-3.14159 upper=3.14159 effort=0.0 velocity=0.0
- added joint Limb3_Limb14: type revolute, parent Limb3, child Limb14, origin xyz=1.1 0 -0.4 rpy=0 0 0, axis 0 1 0, limit lower=-3.14159 upper=3.14159 effort=0.0 velocity=0.0
- added joint Limb6_BotLimb6: type revolute, parent Limb6, child BotLimb6, origin xyz=0 1.4 0 rpy=0 0 0, axis 1 0 0, limit lower=-3.14159 upper=3.14159 effort=0.0 velocity=0.0
- added joint Limb6_Limb12: type revolute, parent Limb6, child Limb12, origin xyz=0.5 0 -0.7 rpy=0 0 0, axis 0 1 0, limit lower=-3.14159 upper=3.14159 effort=0.0 velocity=0.0
- added joint Limb7_BotLimb7: type revolute, parent Limb7, child BotLimb7, origin xyz=0 1.2 0 rpy=0 0 0, axis 1 0 0, limit lower=-3.14159 upper=3.14159 effort=0.0 velocity=0.0
- added joint Limb7_Limb15: type revolute, parent Limb7, child Limb15, origin xyz=0.55 0 -0.6 rpy=0 0 0, axis 0 1 0, limit lower=-3.14159 upper=3.14159 effort=0.0 velocity=0.0
- added joint Limb8_Limb13: type revolute, parent Limb8, child Limb13, origin xyz=0.95 0 -0.4 rpy=0 0 0, axis 0 1 0, limit lower=-3.14159 upper=3.14159 effort=0.0 velocity=0.0
- joint BotLimb0_Limb1: origin xyz=0 1.9 0 rpy=0 0 0 -> xyz=0 2.1 0 rpy=0 0 0
- joint BotLimb1_Limb2: origin xyz=0 1.5 0 rpy=0 0 0 -> xyz=0 1.3 0 rpy=0 0 0
- joint BotLimb2_Limb3: origin xyz=0 1.6 0 rpy=0 0 0 -> xyz=0 1.5 0 rpy=0 0 0
- joint BotLimb3_Limb4: origin xyz=0 1.0 0 rpy=0 0 0 -> xyz=0 0.8 0 rpy=0 0 0
- joint BotLimb4_Limb5: origin xyz=0 1.1 0 rpy=0 0 0 -> xyz=0 1.2 0 rpy=0 0 0
- joint BotLimb5_Limb6: origin xyz=0 1.7 0 rpy=0 0 0 -> xyz=0 2.1 0 rpy=0 0 0
- joint Limb0_BotLimb0: origin xyz=0 0.95 3.1 rpy=0 0 0 -> xyz=0 1.05 2.7 rpy=0 0 0
- joint Limb1_BotLimb1: origin xyz=0 1.5 0 rpy=0 0 0 -> xyz=0 1.3 0 rpy=0 0 0
- joint Limb2_BotLimb2: origin xyz=0 1.6 0 rpy=0 0 0 -> xyz=0 1.5 0 rpy=0 0 0
- joint Limb3_BotLimb3: origin xyz=0 1.0 0 rpy=0 0 0 -> xyz=0 0.8 0 rpy=0 0 0
- joint Limb4_BotLimb4: origin xyz=0 1.1 0 rpy=0 0 0 -> xyz=0 1.2 0 rpy=0 0 0
- joint Limb5_BotLimb5: origin xyz=0 1.7 0 rpy=0 0 0 -> xyz=0 2.1 0 rpy=0 0 0
